Commit message: fifth commit

File: description/gazebo_control.xacro (robot description, xacro)
@@ -3,18 +3,21 @@
     <!-- Controller for the 4-wheeled robot-->
     <gazebo>
-        <plugin name="skid_steer_drive_controller" filename="libgazebo_ros_skid_steer_drive.so">
+        <plugin name="skid_steer_drive_controller" filename="libgazebo_ros_diff_drive.so">
             <!-- Wheel Information -->
-            <!--<left_front_joint>left_front_wheel_joint</left_front_joint>
-            <right_front_joint>right_front_wheel_joint</right_front_joint>
-            <left_rear_joint>left_rear_wheel_joint</left_rear_joint>
-            <right_rear_joint>right_rear_wheel_joint</right_rear_joint>
-            -->
+            <num_wheel_pairs>2</num_wheel_pairs>
             <left_joint>left_front_wheel_joint</left_joint>
+            <left_joint>left_rear_wheel_joint</left_joint>
+            <wheel_separation>0.1785</wheel_separation>
+            <wheel_diameter>0.08</wheel_diameter>
             <right_joint>right_front_wheel_joint</right_joint>
+            <right_joint>right_rear_wheel_joint</right_joint>
+            <wheel_separation>0.1785</wheel_separation>
+            <wheel_diameter>0.08</wheel_diameter>
+            <!--
             <left_joint>left_rear_wheel_joint</left_joint>
             <right_joint>right_rear_wheel_joint</right_joint>
-                            <!-- Distance between left wheel origin and right wheel origin -->
             <wheel_separation>0.1785</wheel_separation>
             <wheel_diameter>0.08</wheel_diameter>
+            -->
             <!-- Limits -->
             <max_wheel_torque>200</max_wheel_torque>

File: description/robot.urdf.xacro (robot description, xacro)
@@ -3,3 +3,5 @@
     <xacro:include filename="robot_core.xacro" />
     <xacro:include filename="gazebo_control.xacro"/>
+    <xacro:include filename="lidar.xacro" />
+    <xacro:include filename="camera.xacro" />
 </robot>

File: description/robot_core.xacro (robot description, xacro)
@@ -40,9 +40,17 @@
         <color rgba="1 0 0 1"/>
     </material>
-    <!-- BASE LINK ************************************************************  -->
+    <!-- BASE LINK *********************************************************  -->
     <!-- Define the center of the main robot chassis projected on the ground -->
     <link name="base_link">
     </link>
-    <!-- CHASSIS **********************************************************  -->
+    <!-- BASE FOOTPRINT ****************************************************  -->
+    <joint name="base_footprint_joint" type="fixed">
+        <parent link="base_link"/>
+        <child link="base_footprint"/>
+        <origin xyz="0 0 0" rpy="0 0 0"/>
+    </joint>
+    <link name="base_footprint">
+    </link>
+    <!-- CHASSIS ***********************************************************  -->
     <joint name="chassis_joint" type="fixed">
         <parent link="base_link"/>
@@ -105,5 +113,5 @@
         <child link="right_front_wheel"/>
         <origin xyz="0.097 -0.068 0" rpy="${pi/2} 0 0"/>
-        <axis xyz="0 0 1"/>
+        <axis xyz="0 0 -1"/>
     </joint>
     <link name="right_front_wheel">
@@ -161,5 +169,5 @@
         <child link="right_rear_wheel"/>
         <origin xyz="0 -0.068 0" rpy="${pi/2} 0 0"/>
-        <axis xyz="0 0 1"/>
+        <axis xyz="0 0 -1"/>
     </joint>
     <link name="right_rear_wheel">
